Commit message: Added object collision to MoveIt planning

File: k1_arm/perception_stack/sagittarius_descriptions/urdf/sgr532.urdf.xacro (robot description, xacro)
@@ -589,8 +589,8 @@
       link="$(arg robot_name)/link_gripper_left" />
     <axis
-      xyz="0 1 0" />
-    <limit
-      lower="-0.034"
-      upper="0"
+      xyz="0 -1 0" />
+    <limit
+      lower="0.0"
+      upper="0.038"
       effort="10"
       velocity="1.14" />
@@ -656,8 +656,8 @@
       link="$(arg robot_name)/link_gripper_right" />
     <axis
-      xyz="0 -1 0" />
-    <limit
-      lower="-0.034"
-      upper="0"
+      xyz="0 1 0" />
+    <limit
+      lower="0"
+      upper="0.038"
       effort="10"
       velocity="1.10" />
